File: Analog.kicad_sch (KiCad schematic)
At the start: 55 parts, among them U10 OPA310xDBV, U11 OPA310xDBV, U12 OPA310xDBV, U13 OPA310xDBV, U14 OPA310xDBV, U15 OPA310xDBV, U16 OPA310xDBV, U17 ADS8688, U9 OPA310xDBV

Commit message: add cap
Parts:
- C80: renamed from C4; footprint (none) -> Capacitor_SMD:C_0603_1608Metric
- C81: renamed from C5; footprint (none) -> Capacitor_SMD:C_0603_1608Metric
- C82: renamed from C6; footprint (none) -> Capacitor_SMD:C_0805_2012Metric
- C83: renamed from C1; footprint (none) -> Capacitor_SMD:C_0805_2012Metric
- C84: renamed from C2; footprint (none) -> Capacitor_SMD:C_0603_1608Metric
- C85: renamed from C3; footprint (none) -> Capacitor_SMD:C_0805_2012Metric
- C86: renamed from C40; value 100nf -> 1uf; footprint Capacitor_SMD:C_0402_1005Metric -> Capacitor_SMD:C_0603_1608Metric
- C87: renamed from C41; value 100nf -> 1uf; footprint Capacitor_SMD:C_0402_1005Metric -> Capacitor_SMD:C_0603_1608Metric
- C88: renamed from C42; value 100nf -> 1uf; footprint Capacitor_SMD:C_0402_1005Metric -> Capacitor_SMD:C_0603_1608Metric
- C89: renamed from C43; value 100nf -> 1uf; footprint Capacitor_SMD:C_0402_1005Metric -> Capacitor_SMD:C_0603_1608Metric
- C90: renamed from C44; value 100nf -> 1uf; footprint Capacitor_SMD:C_0402_1005Metric -> Capacitor_SMD:C_0603_1608Metric
- C91: renamed from C45; value 100nf -> 1uf; footprint Capacitor_SMD:C_0402_1005Metric -> Capacitor_SMD:C_0603_1608Metric
- C92: renamed from C46; value 100nf -> 1uf; footprint Capacitor_SMD:C_0402_1005Metric -> Capacitor_SMD:C_0603_1608Metric
- C93: renamed from C47; value 100nf -> 1uf; footprint Capacitor_SMD:C_0402_1005Metric -> Capacitor_SMD:C_0603_1608Metric
- R10: renamed from R1; footprint (none) -> Resistor_SMD:R_0603_1608Metric
- R11: renamed from R18; footprint (none) -> Resistor_SMD:R_0603_1608Metric
- R12: renamed from R2; footprint (none) -> Resistor_SMD:R_0603_1608Metric
- R13: renamed from R20; footprint (none) -> Resistor_SMD:R_0603_1608Metric
- R14: renamed from R7; footprint (none) -> Resistor_SMD:R_0603_1608Metric
- R15: renamed from R23; footprint (none) -> Resistor_SMD:R_0603_1608Metric
- R16: renamed from R5; footprint (none) -> Resistor_SMD:R_0603_1608Metric
- R17: renamed from R21; footprint (none) -> Resistor_SMD:R_0603_1608Metric
- R18: renamed from R6; footprint (none) -> Resistor_SMD:R_0603_1608Metric
- R19: renamed from R22; footprint (none) -> Resistor_SMD:R_0603_1608Metric
- R20: renamed from R8; footprint (none) -> Resistor_SMD:R_0603_1608Metric
- R21: renamed from R24; footprint (none) -> Resistor_SMD:R_0603_1608Metric
- R22: renamed from R11; footprint (none) -> Resistor_SMD:R_0603_1608Metric
- R23: renamed from R27; footprint (none) -> Resistor_SMD:R_0603_1608Metric
- R24: renamed from R9; footprint (none) -> Resistor_SMD:R_0603_1608Metric
- R25, R31: footprint (none) -> Resistor_SMD:R_0603_1608Metric
- R26: renamed from R10; footprint (none) -> Resistor_SMD:R_0603_1608Metric
- R27: renamed from R26; footprint (none) -> Resistor_SMD:R_0603_1608Metric
- R28: renamed from R12; footprint (none) -> Resistor_SMD:R_0603_1608Metric
- R29: renamed from R28; footprint (none) -> Resistor_SMD:R_0603_1608Metric
- R30: renamed from R15; footprint (none) -> Resistor_SMD:R_0603_1608Metric
- R32: renamed from R13; footprint (none) -> Resistor_SMD:R_0603_1608Metric
- R33: renamed from R29; footprint (none) -> Resistor_SMD:R_0603_1608Metric
- R34: renamed from R14; footprint (none) -> Resistor_SMD:R_0603_1608Metric
- R35: renamed from R30; footprint (none) -> Resistor_SMD:R_0603_1608Metric
- R36: renamed from R16; footprint (none) -> Resistor_SMD:R_0603_1608Metric
- R37: renamed from R32; footprint (none) -> Resistor_SMD:R_0603_1608Metric
- R6: renamed from R4; footprint (none) -> Resistor_SMD:R_0603_1608Metric
- R7: renamed from R19; footprint (none) -> Resistor_SMD:R_0603_1608Metric
- R8: renamed from R3; footprint (none) -> Resistor_SMD:R_0603_1608Metric
- R9: renamed from R17; footprint (none) -> Resistor_SMD:R_0603_1608Metric
- renumbered U9 to U10, U13 to U11, U10 to U12, U14 to U13, U17 to U14, U11 to U15, U15 to U16, U12 to U17, U16 to U18
