File: MW601_KB.kicad_pcb (KiCad board)
At the start: 4 copper layers, 285 x 94.6 mm, 147 parts, among them J1 USB_C_Receptacle_USB2.0_16P, U1 ADG1607xCP, U2 ADG1607xCP, U3 ADG1607xCP, U4 ADG1607xCP, U5 ADG1607xCP, U6 ADG1607xCP, U7 ADG1607xCP, U8 ADG1607xCP

Commit message: sch
Parts:
- added C11: 3.3nf, Capacitor_SMD:C_0603_1608Metric, B.Cu at (161.4, 164.1)
- added C12: 10uf, Capacitor_SMD:C_0603_1608Metric, B.Cu at (161.4, 166.6)
- added C13: 10uf, Capacitor_SMD:C_0603_1608Metric, B.Cu at (161.4, 169.1)
- added C17: 3.3nf, Capacitor_SMD:C_0603_1608Metric, B.Cu at (157.4, 159.0)
- added C18: 10uf, Capacitor_SMD:C_0603_1608Metric, B.Cu at (157.4, 161.5)
- added C34: 100nf, Capacitor_SMD:C_0402_1005Metric, B.Cu at (172.0, 149.6)
- added C35: 12pf, Capacitor_SMD:C_0402_1005Metric, B.Cu at (172.0, 151.6)
- added C36: 12pf, Capacitor_SMD:C_0402_1005Metric, B.Cu at (172.0, 153.6)
- added C37: 100nf, Capacitor_SMD:C_0402_1005Metric, B.Cu at (172.0, 155.5)
- added C38: 100nf, Capacitor_SMD:C_0402_1005Metric, B.Cu at (172.0, 157.5)
- added C39: 100nf, Capacitor_SMD:C_0402_1005Metric, B.Cu at (172.0, 159.5)
- added C40: 100nf, Capacitor_SMD:C_0402_1005Metric, B.Cu at (151.7, 138.3)
- added C41: 100nf, Capacitor_SMD:C_0402_1005Metric, B.Cu at (151.7, 140.2)
- added C42: 100nf, Capacitor_SMD:C_0402_1005Metric, B.Cu at (151.7, 142.2)
- added C43: 100nf, Capacitor_SMD:C_0402_1005Metric, B.Cu at (151.7, 144.2)
- added C44: 100nf, Capacitor_SMD:C_0402_1005Metric, B.Cu at (151.7, 146.1)
- added C45: 100nf, Capacitor_SMD:C_0402_1005Metric, B.Cu at (151.7, 148.1)
- added C46: 100nf, Capacitor_SMD:C_0402_1005Metric, B.Cu at (151.7, 150.1)
- added C47: 100nf, Capacitor_SMD:C_0402_1005Metric, B.Cu at (151.7, 152.1)
- added C7: 10uf, Capacitor_SMD:C_0603_1608Metric, B.Cu at (161.4, 159.0)
- added C8: 3.3nf, Capacitor_SMD:C_0603_1608Metric, B.Cu at (161.4, 161.5)
- added R37: 10k, Resistor_SMD:R_0603_1608Metric, B.Cu at (157.4, 164.1)
- added R40: 309k, Resistor_SMD:R_0603_1608Metric, B.Cu at (157.4, 166.6)
- added R41: 100k, Resistor_SMD:R_0603_1608Metric, B.Cu at (157.4, 169.1)
- added R43: 4.7k, Resistor_SMD:R_0603_1608Metric, B.Cu at (168.5, 149.9)
- added R44: 4.7k, Resistor_SMD:R_0603_1608Metric, B.Cu at (168.5, 152.4)
- added R45: 510R, Resistor_SMD:R_0603_1608Metric, B.Cu at (168.5, 154.9)
- added SW1: SW_SPDT, Button_Switch_THT:SW_Slide_SPDT_Straight_CK_OS102011MS2Q, B.Cu at (181.4, 152.1)
- added SW2: SW_Push, Button_Switch_SMD:SW_Push_1P1T_XKB_TS-1187A, B.Cu at (169.7, 140.6)
- added U10: OPA310xDBV, Package_TO_SOT_SMD:SOT-23-5, B.Cu at (160.9, 139.7)
- added U11: OPA310xDBV, Package_TO_SOT_SMD:SOT-23-5, B.Cu at (160.9, 144.3)
- added U12: OPA310xDBV, Package_TO_SOT_SMD:SOT-23-5, B.Cu at (160.9, 148.9)
- added U13: OPA310xDBV, Package_TO_SOT_SMD:SOT-23-5, B.Cu at (160.9, 153.6)
- added U14: OPA310xDBV, Package_TO_SOT_SMD:SOT-23-5, B.Cu at (155.7, 139.7)
- added U15: OPA310xDBV, Package_TO_SOT_SMD:SOT-23-5, B.Cu at (155.7, 144.3)
- added U16: OPA310xDBV, Package_TO_SOT_SMD:SOT-23-5, B.Cu at (155.7, 148.9)
- added U17: ADS8688, Package_SO:TSSOP-38_4.4x9.7mm_P0.5mm, B.Cu at (143.3, 114.5)
- added U18: TPS82130, Package_LGA:Texas_SIL0008D_MicroSiP-8-1EP_2.8x3mm_P0.65mm_EP1.1x1.9mm_ThermalVias, B.Cu at (153.0, 170.8)
- added U19: TPS74801DRC, Package_SON:VSON-10-1EP_3x3mm_P0.5mm_EP1.65x2.4mm_ThermalVias, B.Cu at (147.9, 126.7)
- added U20: TPS74801DRC, Package_SON:VSON-10-1EP_3x3mm_P0.5mm_EP1.65x2.4mm_ThermalVias, B.Cu at (132.6, 134.2)
- added U21: CH32V30xCxTx, Package_QFP:LQFP-48_7x7mm_P0.5mm, B.Cu at (128.4, 114.7)
- added U9: OPA310xDBV, Package_TO_SOT_SMD:SOT-23-5, B.Cu at (155.7, 154.6)
- added Y1: Crystal_GND24, Crystal:Crystal_SMD_3225-4Pin_3.2x2.5mm, B.Cu at (135.9, 114.3)
- H1, H2, H3, H4, H5, H6: renamed from HOLE; value VAL** -> MountingHole_Pad
- moved U7 160.2 mm to (277.8, 76.5)
- moved U6 133.1 mm to (251.8, 67.4)
- moved U1 96.5 mm to (56.4, 67.4)
- moved U5 95.1 mm to (213.4, 67.4)
- moved U8 74.9 mm to (195.8, 111.1)
- moved U2 66.1 mm to (99.7, 67.4)
- moved U4 64.4 mm to (176.4, 67.4)
- moved U3 42.8 mm to (138.9, 67.5)
- renumbered REF** to H10, REF** to H7, REF** to H8, REF** to H9
Connections:
- net VSSA renamed VCC1V0
- D1 pad 1: VCC_LED -> +5V
- D1 pad 4: LED_SDA -> /Key Layout/LED_SDA
- D10 pad 1: VCC_LED -> +5V
- D11 pad 1: VCC_LED -> +5V
- D12 pad 1: VCC_LED -> +5V
- D13 pad 1: VCC_LED -> +5V
- D14 pad 1: VCC_LED -> +5V
- D15 pad 1: VCC_LED -> +5V
- D16 pad 1: VCC_LED -> +5V
- D17 pad 1: VCC_LED -> +5V
- D18 pad 1: VCC_LED -> +5V
- D19 pad 1: VCC_LED -> +5V
- D2 pad 1: VCC_LED -> +5V
- D20 pad 1: VCC_LED -> +5V
- D21 pad 1: VCC_LED -> +5V
- D22 pad 1: VCC_LED -> +5V
- D23 pad 1: VCC_LED -> +5V
- D24 pad 1: VCC_LED -> +5V
- D25 pad 1: VCC_LED -> +5V
- D26 pad 1: VCC_LED -> +5V
- D27 pad 1: VCC_LED -> +5V
- D28 pad 1: VCC_LED -> +5V
- D29 pad 1: VCC_LED -> +5V
- D3 pad 1: VCC_LED -> +5V
- D30 pad 1: VCC_LED -> +5V
- D31 pad 1: VCC_LED -> +5V
- D32 pad 1: VCC_LED -> +5V
- D33 pad 1: VCC_LED -> +5V
- D34 pad 1: VCC_LED -> +5V
- D35 pad 1: VCC_LED -> +5V
- D36 pad 1: VCC_LED -> +5V
- D37 pad 1: VCC_LED -> +5V
- D38 pad 1: VCC_LED -> +5V
- D39 pad 1: VCC_LED -> +5V
- D4 pad 1: VCC_LED -> +5V
- D40 pad 1: VCC_LED -> +5V
- D41 pad 1: VCC_LED -> +5V
- D42 pad 1: VCC_LED -> +5V
- D43 pad 1: VCC_LED -> +5V
- D44 pad 1: VCC_LED -> +5V
- D45 pad 1: VCC_LED -> +5V
- D46 pad 1: VCC_LED -> +5V
- D47 pad 1: VCC_LED -> +5V
- D48 pad 1: VCC_LED -> +5V
- D49 pad 1: VCC_LED -> +5V
- D5 pad 1: VCC_LED -> +5V
- D50 pad 1: VCC_LED -> +5V
- D51 pad 1: VCC_LED -> +5V
- D52 pad 1: VCC_LED -> +5V
- D53 pad 1: VCC_LED -> +5V
- D54 pad 1: VCC_LED -> +5V
- D55 pad 1: VCC_LED -> +5V
- D56 pad 1: VCC_LED -> +5V
- D57 pad 1: VCC_LED -> +5V
- D58 pad 1: VCC_LED -> +5V
- D59 pad 1: VCC_LED -> +5V
- D6 pad 1: VCC_LED -> +5V
- D60 pad 1: VCC_LED -> +5V
- D61 pad 1: VCC_LED -> +5V
- D62 pad 1: VCC_LED -> +5V
- D63 pad 1: VCC_LED -> +5V
- D64 pad 1: VCC_LED -> +5V
- D7 pad 1: VCC_LED -> +5V
- D8 pad 1: VCC_LED -> +5V
- D9 pad 1: VCC_LED -> +5V
- H1 pad 1: (no net) -> GND
- H2 pad 1: (no net) -> GND
- H3 pad 1: (no net) -> GND
- H4 pad 1: (no net) -> GND
- H5 pad 1: (no net) -> GND
- H6 pad 1: (no net) -> GND
- J1 pad A1: Net-(J1-GND-PadA1) -> GND
- J1 pad A12: Net-(J1-GND-PadA1) -> GND
- J1 pad A4: Net-(J1-VBUS-PadA4) -> +5V
- J1 pad A5: unconnected-(J1-CC1-PadA5) -> Net-(J1-CC1)
- J1 pad A6: unconnected-(J1-D+-PadA6) -> /MCU/D+
- J1 pad A7: unconnected-(J1-D--PadA7) -> /MCU/D-
- J1 pad A9: Net-(J1-VBUS-PadA4) -> +5V
- J1 pad B1: Net-(J1-GND-PadA1) -> GND
- J1 pad B12: Net-(J1-GND-PadA1) -> GND
- J1 pad B4: Net-(J1-VBUS-PadA4) -> +5V
- J1 pad B5: unconnected-(J1-CC2-PadB5) -> Net-(J1-CC2)
- J1 pad B6: unconnected-(J1-D+-PadB6) -> /MCU/D+
- J1 pad B7: unconnected-(J1-D--PadB7) -> /MCU/D-
- J1 pad B9: Net-(J1-VBUS-PadA4) -> +5V
- J1 pad S1: unconnected-(J1-SHIELD-PadS1) -> GND
- MW1 pad 2: OUT_P1 -> /Key Layout/OUT_P1
- MW1 pad 4: OUT_N1 -> /Key Layout/OUT_N1
- MW10 pad 2: OUT_P10 -> /Key Layout/OUT_P10
- MW10 pad 4: OUT_N10 -> /Key Layout/OUT_N10
- MW11 pad 2: OUT_P11 -> /Key Layout/OUT_P11
- MW11 pad 4: OUT_N11 -> /Key Layout/OUT_N11
- MW12 pad 2: OUT_P12 -> /Key Layout/OUT_P12
- MW12 pad 4: OUT_N12 -> /Key Layout/OUT_N12
- MW13 pad 2: OUT_P13 -> /Key Layout/OUT_P13
- MW13 pad 4: OUT_N13 -> /Key Layout/OUT_N13
- MW14 pad 2: OUT_P14 -> /Key Layout/OUT_P14
- MW14 pad 4: OUT_N14 -> /Key Layout/OUT_N14
- MW15 pad 2: OUT_P15 -> /Key Layout/OUT_P15
- MW15 pad 4: OUT_N15 -> /Key Layout/OUT_N15
- MW16 pad 2: OUT_P16 -> /Key Layout/OUT_P16
- MW16 pad 4: OUT_N16 -> /Key Layout/OUT_N16
- MW17 pad 2: OUT_P17 -> /Key Layout/OUT_P17
- MW17 pad 4: OUT_N17 -> /Key Layout/OUT_N17
- MW18 pad 2: OUT_P18 -> /Key Layout/OUT_P18
- MW18 pad 4: OUT_N18 -> /Key Layout/OUT_N18
- MW19 pad 2: OUT_P19 -> /Key Layout/OUT_P19
- MW19 pad 4: OUT_N19 -> /Key Layout/OUT_N19
- MW2 pad 2: OUT_P2 -> /Key Layout/OUT_P2
- MW2 pad 4: OUT_N2 -> /Key Layout/OUT_N2
- MW20 pad 2: OUT_P20 -> /Key Layout/OUT_P20
- MW20 pad 4: OUT_N20 -> /Key Layout/OUT_N20
- MW21 pad 2: OUT_P21 -> /Key Layout/OUT_P21
- MW21 pad 4: OUT_N21 -> /Key Layout/OUT_N21
- MW22 pad 2: OUT_P22 -> /Key Layout/OUT_P22
- MW22 pad 4: OUT_N22 -> /Key Layout/OUT_N22
- MW23 pad 2: OUT_P23 -> /Key Layout/OUT_P23
- MW23 pad 4: OUT_N23 -> /Key Layout/OUT_N23
- MW24 pad 2: OUT_P24 -> /Key Layout/OUT_P24
- MW24 pad 4: OUT_N24 -> /Key Layout/OUT_N24
- MW25 pad 2: OUT_P25 -> /Key Layout/OUT_P25
- MW25 pad 4: OUT_N25 -> /Key Layout/OUT_N25
- MW26 pad 2: OUT_P26 -> /Key Layout/OUT_P26
- MW26 pad 4: OUT_N26 -> /Key Layout/OUT_N26
- MW27 pad 2: OUT_P27 -> /Key Layout/OUT_P27
- MW27 pad 4: OUT_N27 -> /Key Layout/OUT_N27
- MW28 pad 2: OUT_P28 -> /Key Layout/OUT_P28
- MW28 pad 4: OUT_N28 -> /Key Layout/OUT_N28
- MW29 pad 2: OUT_P29 -> /Key Layout/OUT_P29
- MW29 pad 4: OUT_N29 -> /Key Layout/OUT_N29
- MW3 pad 2: OUT_P3 -> /Key Layout/OUT_P3
- MW3 pad 4: OUT_N3 -> /Key Layout/OUT_N3
- MW30 pad 2: OUT_P30 -> /Key Layout/OUT_P30
- MW30 pad 4: OUT_N30 -> /Key Layout/OUT_N30
- MW31 pad 2: OUT_P31 -> /Key Layout/OUT_P31
- MW31 pad 4: OUT_N31 -> /Key Layout/OUT_N31
- MW32 pad 2: OUT_P32 -> /Key Layout/OUT_P32
- MW32 pad 4: OUT_N32 -> /Key Layout/OUT_N32
- MW33 pad 2: OUT_P33 -> /Key Layout/OUT_P33
- MW33 pad 4: OUT_N33 -> /Key Layout/OUT_N33
- MW34 pad 2: OUT_P34 -> /Key Layout/OUT_P34
- MW34 pad 4: OUT_N34 -> /Key Layout/OUT_N34
- MW35 pad 2: OUT_P35 -> /Key Layout/OUT_P35
- MW35 pad 4: OUT_N35 -> /Key Layout/OUT_N35
- MW36 pad 2: OUT_P36 -> /Key Layout/OUT_P36
- MW36 pad 4: OUT_N36 -> /Key Layout/OUT_N36
- MW37 pad 2: OUT_P37 -> /Key Layout/OUT_P37
- MW37 pad 4: OUT_N37 -> /Key Layout/OUT_N37
- MW38 pad 2: OUT_P38 -> /Key Layout/OUT_P38
- MW38 pad 4: OUT_N38 -> /Key Layout/OUT_N38
- MW39 pad 2: OUT_P39 -> /Key Layout/OUT_P39
- MW39 pad 4: OUT_N39 -> /Key Layout/OUT_N39
- MW4 pad 2: OUT_P4 -> /Key Layout/OUT_P4
- MW4 pad 4: OUT_N4 -> /Key Layout/OUT_N4
- MW40 pad 2: OUT_P40 -> /Key Layout/OUT_P40
- MW40 pad 4: OUT_N40 -> /Key Layout/OUT_N40
- MW41 pad 2: OUT_P41 -> /Key Layout/OUT_P41
- MW41 pad 4: OUT_N41 -> /Key Layout/OUT_N41
- MW42 pad 2: OUT_P42 -> /Key Layout/OUT_P42
- MW42 pad 4: OUT_N42 -> /Key Layout/OUT_N42
- MW43 pad 2: OUT_P43 -> /Key Layout/OUT_P43
- MW43 pad 4: OUT_N43 -> /Key Layout/OUT_N43
- MW44 pad 2: OUT_P44 -> /Key Layout/OUT_P44
- MW44 pad 4: OUT_N44 -> /Key Layout/OUT_N44
- MW45 pad 2: OUT_P45 -> /Key Layout/OUT_P45
- MW45 pad 4: OUT_N45 -> /Key Layout/OUT_N45
- MW46 pad 2: OUT_P46 -> /Key Layout/OUT_P46
- MW46 pad 4: OUT_N46 -> /Key Layout/OUT_N46
- MW47 pad 2: OUT_P47 -> /Key Layout/OUT_P47
- MW47 pad 4: OUT_N47 -> /Key Layout/OUT_N47
- MW48 pad 2: OUT_P48 -> /Key Layout/OUT_P48
- MW48 pad 4: OUT_N48 -> /Key Layout/OUT_N48
- MW49 pad 2: OUT_P49 -> /Key Layout/OUT_P49
- MW49 pad 4: OUT_N49 -> /Key Layout/OUT_N49
- MW5 pad 2: OUT_P5 -> /Key Layout/OUT_P5
- MW5 pad 4: OUT_N5 -> /Key Layout/OUT_N5
- MW50 pad 2: OUT_P50 -> /Key Layout/OUT_P50
- MW50 pad 4: OUT_N50 -> /Key Layout/OUT_N50
- MW51 pad 2: OUT_P51 -> /Key Layout/OUT_P51
- MW51 pad 4: OUT_N51 -> /Key Layout/OUT_N51
- MW52 pad 2: OUT_P52 -> /Key Layout/OUT_P52
- MW52 pad 4: OUT_N52 -> /Key Layout/OUT_N52
- MW53 pad 2: OUT_P53 -> /Key Layout/OUT_P53
- MW53 pad 4: OUT_N53 -> /Key Layout/OUT_N53
- MW54 pad 2: OUT_P54 -> /Key Layout/OUT_P54
- MW54 pad 4: OUT_N54 -> /Key Layout/OUT_N54
- MW55 pad 2: OUT_P55 -> /Key Layout/OUT_P55
- MW55 pad 4: OUT_N55 -> /Key Layout/OUT_N55
- MW56 pad 2: OUT_P56 -> /Key Layout/OUT_P56
- MW56 pad 4: OUT_N56 -> /Key Layout/OUT_N56
- MW57 pad 2: OUT_P57 -> /Key Layout/OUT_P57
- MW57 pad 4: OUT_N57 -> /Key Layout/OUT_N57
- MW58 pad 2: OUT_P58 -> /Key Layout/OUT_P58
- MW58 pad 4: OUT_N58 -> /Key Layout/OUT_N58
- MW59 pad 2: OUT_P59 -> /Key Layout/OUT_P59
- MW59 pad 4: OUT_N59 -> /Key Layout/OUT_N59
- MW6 pad 2: OUT_P6 -> /Key Layout/OUT_P6
- MW6 pad 4: OUT_N6 -> /Key Layout/OUT_N6
- MW60 pad 2: OUT_P60 -> /Key Layout/OUT_P60
- MW60 pad 4: OUT_N60 -> /Key Layout/OUT_N60
- MW61 pad 2: OUT_P61 -> /Key Layout/OUT_P61
- MW61 pad 4: OUT_N61 -> /Key Layout/OUT_N61
- MW62 pad 2: OUT_P62 -> /Key Layout/OUT_P62
- MW62 pad 4: OUT_N62 -> /Key Layout/OUT_N62
- MW63 pad 2: OUT_P63 -> /Key Layout/OUT_P63
- MW63 pad 4: OUT_N63 -> /Key Layout/OUT_N63
- MW64 pad 2: OUT_P64 -> /Key Layout/OUT_P64
- MW64 pad 4: OUT_N64 -> /Key Layout/OUT_N64
- MW7 pad 2: OUT_P7 -> /Key Layout/OUT_P7
- MW7 pad 4: OUT_N7 -> /Key Layout/OUT_N7
- MW8 pad 2: OUT_P8 -> /Key Layout/OUT_P8
- MW8 pad 4: OUT_N8 -> /Key Layout/OUT_N8
- MW9 pad 2: OUT_P9 -> /Key Layout/OUT_P9
- MW9 pad 4: OUT_N9 -> /Key Layout/OUT_N9
- U1 pad 1: unconnected-(U1-S8B-Pad1) -> /Key Layout/OUT_N43
- U1 pad 10: unconnected-(U1-A2-Pad10) -> /MCU/A2
- U1 pad 14: unconnected-(U1-A1-Pad14) -> /MCU/A1
- U1 pad 15: unconnected-(U1-A0-Pad15) -> /MCU/A0
- U1 pad 16: unconnected-(U1-EN-Pad16) -> /MCU/EN
- U1 pad 17: unconnected-(U1-S1A-Pad17) -> /Key Layout/OUT_P1
- U1 pad 18: unconnected-(U1-S2A-Pad18) -> /Key Layout/OUT_P2
- U1 pad 19: unconnected-(U1-S3A-Pad19) -> /Key Layout/OUT_P15
- U1 pad 2: unconnected-(U1-S7B-Pad2) -> /Key Layout/OUT_N42
- U1 pad 20: unconnected-(U1-S4A-Pad20) -> /Key Layout/OUT_P16
- U1 pad 21: unconnected-(U1-S5A-Pad21) -> /Key Layout/OUT_P29
- U1 pad 22: unconnected-(U1-S6A-Pad22) -> /Key Layout/OUT_P30
- U1 pad 23: unconnected-(U1-S7A-Pad23) -> /Key Layout/OUT_P42
- U1 pad 24: unconnected-(U1-S8A-Pad24) -> /Key Layout/OUT_P43
- U1 pad 27: unconnected-(U1-DA-Pad27) -> /Analog/GP0_OUT+
- U1 pad 3: unconnected-(U1-S6B-Pad3) -> /Key Layout/OUT_N30
- U1 pad 31: unconnected-(U1-DB-Pad31) -> /Analog/GP0_OUT-
- U1 pad 4: unconnected-(U1-S5B-Pad4) -> /Key Layout/OUT_N29
- U1 pad 5: unconnected-(U1-S4B-Pad5) -> /Key Layout/OUT_N16
- U1 pad 6: unconnected-(U1-S3B-Pad6) -> /Key Layout/OUT_N15
- U1 pad 7: unconnected-(U1-S2B-Pad7) -> /Key Layout/OUT_N2
- U1 pad 8: unconnected-(U1-S1B-Pad8) -> /Key Layout/OUT_N1
- U2 pad 1: unconnected-(U2-S8B-Pad1) -> /Key Layout/OUT_N45
- U2 pad 10: unconnected-(U2-A2-Pad10) -> /MCU/A2
- U2 pad 14: unconnected-(U2-A1-Pad14) -> /MCU/A1
- U2 pad 15: unconnected-(U2-A0-Pad15) -> /MCU/A0
- U2 pad 16: unconnected-(U2-EN-Pad16) -> /MCU/EN
- U2 pad 17: unconnected-(U2-S1A-Pad17) -> /Key Layout/OUT_P3
- U2 pad 18: unconnected-(U2-S2A-Pad18) -> /Key Layout/OUT_P4
- U2 pad 19: unconnected-(U2-S3A-Pad19) -> /Key Layout/OUT_P17
- U2 pad 2: unconnected-(U2-S7B-Pad2) -> /Key Layout/OUT_N44
- U2 pad 20: unconnected-(U2-S4A-Pad20) -> /Key Layout/OUT_P18
- U2 pad 21: unconnected-(U2-S5A-Pad21) -> /Key Layout/OUT_P31
- U2 pad 22: unconnected-(U2-S6A-Pad22) -> /Key Layout/OUT_P32
- U2 pad 23: unconnected-(U2-S7A-Pad23) -> /Key Layout/OUT_P44
- U2 pad 24: unconnected-(U2-S8A-Pad24) -> /Key Layout/OUT_P45
- U2 pad 27: unconnected-(U2-DA-Pad27) -> /Analog/GP1_OUT+
- U2 pad 3: unconnected-(U2-S6B-Pad3) -> /Key Layout/OUT_N32
- U2 pad 31: unconnected-(U2-DB-Pad31) -> /Analog/GP1_OUT-
- U2 pad 4: unconnected-(U2-S5B-Pad4) -> /Key Layout/OUT_N31
- U2 pad 5: unconnected-(U2-S4B-Pad5) -> /Key Layout/OUT_N18
- U2 pad 6: unconnected-(U2-S3B-Pad6) -> /Key Layout/OUT_N17
- U2 pad 7: unconnected-(U2-S2B-Pad7) -> /Key Layout/OUT_N4
- U2 pad 8: unconnected-(U2-S1B-Pad8) -> /Key Layout/OUT_N3
- U3 pad 1: unconnected-(U3-S8B-Pad1) -> /Key Layout/OUT_N47
- U3 pad 10: unconnected-(U3-A2-Pad10) -> /MCU/A2
- U3 pad 14: unconnected-(U3-A1-Pad14) -> /MCU/A1
- U3 pad 15: unconnected-(U3-A0-Pad15) -> /MCU/A0
- U3 pad 16: unconnected-(U3-EN-Pad16) -> /MCU/EN
- U3 pad 17: unconnected-(U3-S1A-Pad17) -> /Key Layout/OUT_P5
- U3 pad 18: unconnected-(U3-S2A-Pad18) -> /Key Layout/OUT_P6
- U3 pad 19: unconnected-(U3-S3A-Pad19) -> /Key Layout/OUT_P19
- U3 pad 2: unconnected-(U3-S7B-Pad2) -> /Key Layout/OUT_N46
- U3 pad 20: unconnected-(U3-S4A-Pad20) -> /Key Layout/OUT_P20
- U3 pad 21: unconnected-(U3-S5A-Pad21) -> /Key Layout/OUT_P33
- U3 pad 22: unconnected-(U3-S6A-Pad22) -> /Key Layout/OUT_P34
- U3 pad 23: unconnected-(U3-S7A-Pad23) -> /Key Layout/OUT_P46
- U3 pad 24: unconnected-(U3-S8A-Pad24) -> /Key Layout/OUT_P47
- U3 pad 27: unconnected-(U3-DA-Pad27) -> /Analog/GP2_OUT+
- U3 pad 3: unconnected-(U3-S6B-Pad3) -> /Key Layout/OUT_N34
- U3 pad 31: unconnected-(U3-DB-Pad31) -> /Analog/GP2_OUT-
- U3 pad 4: unconnected-(U3-S5B-Pad4) -> /Key Layout/OUT_N33
- U3 pad 5: unconnected-(U3-S4B-Pad5) -> /Key Layout/OUT_N20
- U3 pad 6: unconnected-(U3-S3B-Pad6) -> /Key Layout/OUT_N19
- U3 pad 7: unconnected-(U3-S2B-Pad7) -> /Key Layout/OUT_N6
- U3 pad 8: unconnected-(U3-S1B-Pad8) -> /Key Layout/OUT_N5
- U4 pad 1: unconnected-(U4-S8B-Pad1) -> /Key Layout/OUT_N49
- U4 pad 10: unconnected-(U4-A2-Pad10) -> /MCU/A2
- U4 pad 14: unconnected-(U4-A1-Pad14) -> /MCU/A1
- U4 pad 15: unconnected-(U4-A0-Pad15) -> /MCU/A0
- U4 pad 16: unconnected-(U4-EN-Pad16) -> /MCU/EN
- U4 pad 17: unconnected-(U4-S1A-Pad17) -> /Key Layout/OUT_P7
- U4 pad 18: unconnected-(U4-S2A-Pad18) -> /Key Layout/OUT_P8
- U4 pad 19: unconnected-(U4-S3A-Pad19) -> /Key Layout/OUT_P21
- U4 pad 2: unconnected-(U4-S7B-Pad2) -> /Key Layout/OUT_N48
- U4 pad 20: unconnected-(U4-S4A-Pad20) -> /Key Layout/OUT_P22
- U4 pad 21: unconnected-(U4-S5A-Pad21) -> /Key Layout/OUT_P35
- U4 pad 22: unconnected-(U4-S6A-Pad22) -> /Key Layout/OUT_P36
- U4 pad 23: unconnected-(U4-S7A-Pad23) -> /Key Layout/OUT_P48
- U4 pad 24: unconnected-(U4-S8A-Pad24) -> /Key Layout/OUT_P49
- U4 pad 27: unconnected-(U4-DA-Pad27) -> /Analog/GP3_OUT+
- U4 pad 3: unconnected-(U4-S6B-Pad3) -> /Key Layout/OUT_N36
- U4 pad 31: unconnected-(U4-DB-Pad31) -> /Analog/GP3_OUT-
- U4 pad 4: unconnected-(U4-S5B-Pad4) -> /Key Layout/OUT_N35
- U4 pad 5: unconnected-(U4-S4B-Pad5) -> /Key Layout/OUT_N22
- U4 pad 6: unconnected-(U4-S3B-Pad6) -> /Key Layout/OUT_N21
- U4 pad 7: unconnected-(U4-S2B-Pad7) -> /Key Layout/OUT_N8
- U4 pad 8: unconnected-(U4-S1B-Pad8) -> /Key Layout/OUT_N7
- U5 pad 1: unconnected-(U5-S8B-Pad1) -> /Key Layout/OUT_N51
- U5 pad 10: unconnected-(U5-A2-Pad10) -> /MCU/A2
- U5 pad 14: unconnected-(U5-A1-Pad14) -> /MCU/A1
- U5 pad 15: unconnected-(U5-A0-Pad15) -> /MCU/A0
- U5 pad 16: unconnected-(U5-EN-Pad16) -> /MCU/EN
- U5 pad 17: unconnected-(U5-S1A-Pad17) -> /Key Layout/OUT_P9
- U5 pad 18: unconnected-(U5-S2A-Pad18) -> /Key Layout/OUT_P10
- U5 pad 19: unconnected-(U5-S3A-Pad19) -> /Key Layout/OUT_P23
- U5 pad 2: unconnected-(U5-S7B-Pad2) -> /Key Layout/OUT_N50
- U5 pad 20: unconnected-(U5-S4A-Pad20) -> /Key Layout/OUT_P24
- U5 pad 21: unconnected-(U5-S5A-Pad21) -> /Key Layout/OUT_P37
- U5 pad 22: unconnected-(U5-S6A-Pad22) -> /Key Layout/OUT_P38
- U5 pad 23: unconnected-(U5-S7A-Pad23) -> /Key Layout/OUT_P50
- U5 pad 24: unconnected-(U5-S8A-Pad24) -> /Key Layout/OUT_P51
- U5 pad 27: unconnected-(U5-DA-Pad27) -> /Analog/GP4_OUT+
- U5 pad 3: unconnected-(U5-S6B-Pad3) -> /Key Layout/OUT_N38
- U5 pad 31: unconnected-(U5-DB-Pad31) -> /Analog/GP4_OUT-
- U5 pad 4: unconnected-(U5-S5B-Pad4) -> /Key Layout/OUT_N37
- U5 pad 5: unconnected-(U5-S4B-Pad5) -> /Key Layout/OUT_N24
- U5 pad 6: unconnected-(U5-S3B-Pad6) -> /Key Layout/OUT_N23
- U5 pad 7: unconnected-(U5-S2B-Pad7) -> /Key Layout/OUT_N10
- U5 pad 8: unconnected-(U5-S1B-Pad8) -> /Key Layout/OUT_N9
- U6 pad 1: unconnected-(U6-S8B-Pad1) -> /Key Layout/OUT_N53
- U6 pad 10: unconnected-(U6-A2-Pad10) -> /MCU/A2
- U6 pad 14: unconnected-(U6-A1-Pad14) -> /MCU/A1
- U6 pad 15: unconnected-(U6-A0-Pad15) -> /MCU/A0
- U6 pad 16: unconnected-(U6-EN-Pad16) -> /MCU/EN
- U6 pad 17: unconnected-(U6-S1A-Pad17) -> /Key Layout/OUT_P11
- U6 pad 18: unconnected-(U6-S2A-Pad18) -> /Key Layout/OUT_P12
- U6 pad 19: unconnected-(U6-S3A-Pad19) -> /Key Layout/OUT_P25
- U6 pad 2: unconnected-(U6-S7B-Pad2) -> /Key Layout/OUT_N52
- U6 pad 20: unconnected-(U6-S4A-Pad20) -> /Key Layout/OUT_P26
- U6 pad 21: unconnected-(U6-S5A-Pad21) -> /Key Layout/OUT_P39
- U6 pad 22: unconnected-(U6-S6A-Pad22) -> /Key Layout/OUT_P40
- U6 pad 23: unconnected-(U6-S7A-Pad23) -> /Key Layout/OUT_P52
- U6 pad 24: unconnected-(U6-S8A-Pad24) -> /Key Layout/OUT_P53
- U6 pad 27: unconnected-(U6-DA-Pad27) -> /Analog/GP5_OUT+
- U6 pad 3: unconnected-(U6-S6B-Pad3) -> /Key Layout/OUT_N40
- U6 pad 31: unconnected-(U6-DB-Pad31) -> /Analog/GP5_OUT-
- U6 pad 4: unconnected-(U6-S5B-Pad4) -> /Key Layout/OUT_N39
- U6 pad 5: unconnected-(U6-S4B-Pad5) -> /Key Layout/OUT_N26
- U6 pad 6: unconnected-(U6-S3B-Pad6) -> /Key Layout/OUT_N25
- U6 pad 7: unconnected-(U6-S2B-Pad7) -> /Key Layout/OUT_N12
- U6 pad 8: unconnected-(U6-S1B-Pad8) -> /Key Layout/OUT_N11
- U7 pad 1: unconnected-(U7-S8B-Pad1) -> /Key Layout/OUT_N64
- U7 pad 10: unconnected-(U7-A2-Pad10) -> /MCU/A2
- U7 pad 14: unconnected-(U7-A1-Pad14) -> /MCU/A1
- U7 pad 15: unconnected-(U7-A0-Pad15) -> /MCU/A0
- U7 pad 16: unconnected-(U7-EN-Pad16) -> /MCU/EN
- U7 pad 17: unconnected-(U7-S1A-Pad17) -> /Key Layout/OUT_P13
- U7 pad 18: unconnected-(U7-S2A-Pad18) -> /Key Layout/OUT_P14
- U7 pad 19: unconnected-(U7-S3A-Pad19) -> /Key Layout/OUT_P27
- U7 pad 2: unconnected-(U7-S7B-Pad2) -> /Key Layout/OUT_N55
- U7 pad 20: unconnected-(U7-S4A-Pad20) -> /Key Layout/OUT_P28
- U7 pad 21: unconnected-(U7-S5A-Pad21) -> /Key Layout/OUT_P41
- U7 pad 22: unconnected-(U7-S6A-Pad22) -> /Key Layout/OUT_P54
- U7 pad 23: unconnected-(U7-S7A-Pad23) -> /Key Layout/OUT_P55
- U7 pad 24: unconnected-(U7-S8A-Pad24) -> /Key Layout/OUT_P64
- U7 pad 27: unconnected-(U7-DA-Pad27) -> /Analog/GP6_OUT+
- U7 pad 3: unconnected-(U7-S6B-Pad3) -> /Key Layout/OUT_N54
- U7 pad 31: unconnected-(U7-DB-Pad31) -> /Analog/GP6_OUT-
- U7 pad 4: unconnected-(U7-S5B-Pad4) -> /Key Layout/OUT_N41
- U7 pad 5: unconnected-(U7-S4B-Pad5) -> /Key Layout/OUT_N28
- U7 pad 6: unconnected-(U7-S3B-Pad6) -> /Key Layout/OUT_N27
- U7 pad 7: unconnected-(U7-S2B-Pad7) -> /Key Layout/OUT_N14
- U7 pad 8: unconnected-(U7-S1B-Pad8) -> /Key Layout/OUT_N13
- U8 pad 1: unconnected-(U8-S8B-Pad1) -> /Key Layout/OUT_N63
- U8 pad 10: unconnected-(U8-A2-Pad10) -> /MCU/A2
- U8 pad 14: unconnected-(U8-A1-Pad14) -> /MCU/A1
- U8 pad 15: unconnected-(U8-A0-Pad15) -> /MCU/A0
- U8 pad 16: unconnected-(U8-EN-Pad16) -> /MCU/EN
- U8 pad 17: unconnected-(U8-S1A-Pad17) -> /Key Layout/OUT_P56
- U8 pad 18: unconnected-(U8-S2A-Pad18) -> /Key Layout/OUT_P57
- U8 pad 19: unconnected-(U8-S3A-Pad19) -> /Key Layout/OUT_P58
- U8 pad 2: unconnected-(U8-S7B-Pad2) -> /Key Layout/OUT_N62
- U8 pad 20: unconnected-(U8-S4A-Pad20) -> /Key Layout/OUT_P59
- U8 pad 21: unconnected-(U8-S5A-Pad21) -> /Key Layout/OUT_P60
- U8 pad 22: unconnected-(U8-S6A-Pad22) -> /Key Layout/OUT_P61
- U8 pad 23: unconnected-(U8-S7A-Pad23) -> /Key Layout/OUT_P62
- U8 pad 24: unconnected-(U8-S8A-Pad24) -> /Key Layout/OUT_P63
- U8 pad 27: unconnected-(U8-DA-Pad27) -> /Analog/GP7_OUT+
- U8 pad 3: unconnected-(U8-S6B-Pad3) -> /Key Layout/OUT_N61
- U8 pad 31: unconnected-(U8-DB-Pad31) -> /Analog/GP7_OUT-
- U8 pad 4: unconnected-(U8-S5B-Pad4) -> /Key Layout/OUT_N60
- U8 pad 5: unconnected-(U8-S4B-Pad5) -> /Key Layout/OUT_N59
- U8 pad 6: unconnected-(U8-S3B-Pad6) -> /Key Layout/OUT_N58
- U8 pad 7: unconnected-(U8-S2B-Pad7) -> /Key Layout/OUT_N57
- U8 pad 8: unconnected-(U8-S1B-Pad8) -> /Key Layout/OUT_N56
Routing:
- added copper zone on In1.Cu, net GND

Commit message: add cap
Parts:
- removed the SW1 at (181.4, 152.1)
- added C1: 1uf, Capacitor_SMD:C_0603_1608Metric, B.Cu at (41.1, 38.1)
- added C10: 1uf, Capacitor_SMD:C_0603_1608Metric, B.Cu at (212.6, 38.1)
- added C100: 1uf, Capacitor_SMD:C_0603_1608Metric, B.Cu at (160.8, 66.3)
- added C101: 100nf, Capacitor_SMD:C_0603_1608Metric, B.Cu at (160.8, 63.2)
- added C103: 22uf, Capacitor_SMD:C_0805_2012Metric, B.Cu at (152.1, 58.2)
- added C104: 1uf, Capacitor_SMD:C_0603_1608Metric, B.Cu at (151.9, 62.1)
- added C105: 100nf, Capacitor_SMD:C_0603_1608Metric, B.Cu at (151.9, 63.6)
- added C107: 1uf, Capacitor_SMD:C_0603_1608Metric, B.Cu at (157.2, 46.6)
- added C108: 4.7uf, Capacitor_SMD:C_0603_1608Metric, B.Cu at (157.2, 48.1)
- added C11: 1uf, Capacitor_SMD:C_0603_1608Metric, B.Cu at (231.6, 38.1)
- added C110: 22uf, Capacitor_SMD:C_0805_2012Metric, B.Cu at (146.9, 44.9)
- added C12: 1uf, Capacitor_SMD:C_0603_1608Metric, B.Cu at (250.7, 38.1)
- added C13: 1uf, Capacitor_SMD:C_0603_1608Metric, B.Cu at (269.7, 38.1)
- added C14: 1uf, Capacitor_SMD:C_0603_1608Metric, B.Cu at (298.3, 38.1)
- added C15: 1uf, Capacitor_SMD:C_0603_1608Metric, B.Cu at (45.9, 57.1)
- added C16: 1uf, Capacitor_SMD:C_0603_1608Metric, B.Cu at (69.7, 57.1)
- added C17: 1uf, Capacitor_SMD:C_0603_1608Metric, B.Cu at (88.7, 57.1)
- added C18: 1uf, Capacitor_SMD:C_0603_1608Metric, B.Cu at (107.8, 57.1)
- added C19: 1uf, Capacitor_SMD:C_0603_1608Metric, B.Cu at (126.8, 57.1)
- added C2: 1uf, Capacitor_SMD:C_0603_1608Metric, B.Cu at (60.1, 38.1)
- added C20: 1uf, Capacitor_SMD:C_0603_1608Metric, B.Cu at (145.9, 57.1)
- added C21: 1uf, Capacitor_SMD:C_0603_1608Metric, B.Cu at (164.9, 57.1)
- added C22: 1uf, Capacitor_SMD:C_0603_1608Metric, B.Cu at (184.0, 57.1)
- added C23: 1uf, Capacitor_SMD:C_0603_1608Metric, B.Cu at (203.0, 57.1)
- added C24: 1uf, Capacitor_SMD:C_0603_1608Metric, B.Cu at (222.1, 57.1)
- added C25: 1uf, Capacitor_SMD:C_0603_1608Metric, B.Cu at (241.1, 57.1)
- added C26: 1uf, Capacitor_SMD:C_0603_1608Metric, B.Cu at (260.2, 57.1)
- added C27: 1uf, Capacitor_SMD:C_0603_1608Metric, B.Cu at (279.2, 57.1)
- added C28: 1uf, Capacitor_SMD:C_0603_1608Metric, B.Cu at (303.0, 57.1)
- added C29: 1uf, Capacitor_SMD:C_0603_1608Metric, B.Cu at (48.2, 76.2)
- added C3: 1uf, Capacitor_SMD:C_0603_1608Metric, B.Cu at (79.2, 38.1)
- added C30: 1uf, Capacitor_SMD:C_0603_1608Metric, B.Cu at (74.4, 76.2)
- added C31: 1uf, Capacitor_SMD:C_0603_1608Metric, B.Cu at (93.5, 76.2)
- added C32: 1uf, Capacitor_SMD:C_0603_1608Metric, B.Cu at (112.5, 76.2)
- added C33: 1uf, Capacitor_SMD:C_0603_1608Metric, B.Cu at (131.6, 76.2)
- added C34: 1uf, Capacitor_SMD:C_0603_1608Metric, B.Cu at (150.6, 76.2)
- added C35: 1uf, Capacitor_SMD:C_0603_1608Metric, B.Cu at (169.7, 76.2)
- added C36: 1uf, Capacitor_SMD:C_0603_1608Metric, B.Cu at (188.7, 76.2)
- added C37: 1uf, Capacitor_SMD:C_0603_1608Metric, B.Cu at (207.8, 76.2)
- added C38: 1uf, Capacitor_SMD:C_0603_1608Metric, B.Cu at (226.8, 76.2)
- added C39: 1uf, Capacitor_SMD:C_0603_1608Metric, B.Cu at (245.9, 76.2)
- added C4: 1uf, Capacitor_SMD:C_0603_1608Metric, B.Cu at (98.2, 38.1)
- added C40: 1uf, Capacitor_SMD:C_0603_1608Metric, B.Cu at (264.9, 76.2)
- added C41: 1uf, Capacitor_SMD:C_0603_1608Metric, B.Cu at (295.9, 76.2)
- added C42: 1uf, Capacitor_SMD:C_0603_1608Metric, B.Cu at (50.6, 95.2)
- added C43: 1uf, Capacitor_SMD:C_0603_1608Metric, B.Cu at (79.2, 95.2)
- added C44: 1uf, Capacitor_SMD:C_0603_1608Metric, B.Cu at (98.2, 95.2)
- added C45: 1uf, Capacitor_SMD:C_0603_1608Metric, B.Cu at (117.3, 95.2)
- added C46: 1uf, Capacitor_SMD:C_0603_1608Metric, B.Cu at (136.3, 95.2)
- added C47: 1uf, Capacitor_SMD:C_0603_1608Metric, B.Cu at (155.4, 95.2)
- added C48: 1uf, Capacitor_SMD:C_0603_1608Metric, B.Cu at (174.4, 95.2)
- added C49: 1uf, Capacitor_SMD:C_0603_1608Metric, B.Cu at (193.5, 95.2)
- added C5: 1uf, Capacitor_SMD:C_0603_1608Metric, B.Cu at (117.3, 38.1)
- added C50: 1uf, Capacitor_SMD:C_0603_1608Metric, B.Cu at (212.6, 95.2)
- added C51: 1uf, Capacitor_SMD:C_0603_1608Metric, B.Cu at (231.6, 95.2)
- added C52: 1uf, Capacitor_SMD:C_0603_1608Metric, B.Cu at (250.7, 95.2)
- added C53: 1uf, Capacitor_SMD:C_0603_1608Metric, B.Cu at (269.7, 95.2)
- added C54: 1uf, Capacitor_SMD:C_0603_1608Metric, B.Cu at (288.8, 95.2)
- added C55: 1uf, Capacitor_SMD:C_0603_1608Metric, B.Cu at (307.8, 95.2)
- added C56: 1uf, Capacitor_SMD:C_0603_1608Metric, B.Cu at (43.5, 114.3)
- added C57: 1uf, Capacitor_SMD:C_0603_1608Metric, B.Cu at (67.3, 114.3)
- added C58: 1uf, Capacitor_SMD:C_0603_1608Metric, B.Cu at (91.1, 114.3)
- added C59: 1uf, Capacitor_SMD:C_0603_1608Metric, B.Cu at (162.5, 114.3)
- added C6: 1uf, Capacitor_SMD:C_0603_1608Metric, B.Cu at (136.3, 38.1)
- added C60: 1uf, Capacitor_SMD:C_0603_1608Metric, B.Cu at (231.6, 114.3)
- added C61: 1uf, Capacitor_SMD:C_0603_1608Metric, B.Cu at (250.7, 114.3)
- added C62: 1uf, Capacitor_SMD:C_0603_1608Metric, B.Cu at (269.7, 114.3)
- added C63: 1uf, Capacitor_SMD:C_0603_1608Metric, B.Cu at (288.8, 114.3)
- added C64: 1uf, Capacitor_SMD:C_0603_1608Metric, B.Cu at (307.8, 114.3)
- added C65: 47uf, Capacitor_SMD:C_0805_2012Metric, B.Cu at (228.4, 132.8)
- added C66: 47uf, Capacitor_SMD:C_0805_2012Metric, B.Cu at (228.4, 135.8)
- added C67: 47uf, Capacitor_SMD:C_0805_2012Metric, B.Cu at (228.4, 138.8)
- added C68: 47uf, Capacitor_SMD:C_0805_2012Metric, B.Cu at (228.4, 141.8)
- added C69: 47uf, Capacitor_SMD:C_0805_2012Metric, B.Cu at (228.4, 144.9)
- added C7: 1uf, Capacitor_SMD:C_0603_1608Metric, B.Cu at (155.4, 38.1)
- added C70: 47uf, Capacitor_SMD:C_0805_2012Metric, B.Cu at (228.4, 147.9)
- added C71: 47uf, Capacitor_SMD:C_0805_2012Metric, B.Cu at (228.4, 150.9)
- added C72: 47uf, Capacitor_SMD:C_0805_2012Metric, B.Cu at (228.4, 153.9)
- added C77: 47uf Polarized, Capacitor_Tantalum_SMD:CP_EIA-3528-21_Kemet-B, B.Cu at (47.6, 41.6)
- added C8: 1uf, Capacitor_SMD:C_0603_1608Metric, B.Cu at (174.4, 38.1)
- added C80: 1uf, Capacitor_SMD:C_0603_1608Metric, B.Cu at (107.2, 146.7)
- added C81: 1uf, Capacitor_SMD:C_0603_1608Metric, B.Cu at (107.2, 149.2)
- added C82: 10uf, Capacitor_SMD:C_0805_2012Metric, B.Cu at (205.9, 132.8)
- added C83: 10uf, Capacitor_SMD:C_0805_2012Metric, B.Cu at (205.9, 135.8)
- added C84: 1uf, Capacitor_SMD:C_0603_1608Metric, B.Cu at (107.2, 151.8)
- added C85: 22uf, Capacitor_SMD:C_0805_2012Metric, B.Cu at (205.9, 138.8)
- added C9: 1uf, Capacitor_SMD:C_0603_1608Metric, B.Cu at (193.5, 38.1)
- added C97: 1uf, Capacitor_SMD:C_0603_1608Metric, B.Cu at (160.8, 64.8)
- added C98: 47uf, Capacitor_SMD:C_0805_2012Metric, B.Cu at (161.0, 61.4)
- added C99: 10uf, Capacitor_SMD:C_0805_2012Metric, B.Cu at (161.0, 68.2)
- added D65: LED, LED_SMD:LED_0603_1608Metric, B.Cu at (191.0, 144.2)
- added J1: Conn_01x06, Connector_PinHeader_2.54mm:PinHeader_1x06_P2.54mm_Vertical, B.Cu at (99.2, 107.7)
- added J3: Boot0, Connector_PinHeader_2.54mm:PinHeader_1x02_P2.54mm_Vertical, B.Cu at (54.7, 76.8)
- added R10: 1k, Resistor_SMD:R_0603_1608Metric, B.Cu at (61.6, 65.7)
- added R11: 1k, Resistor_SMD:R_0603_1608Metric, B.Cu at (222.2, 145.1)
- added R12: 6k, Resistor_SMD:R_0603_1608Metric, B.Cu at (64.9, 64.0)
- added R13: 6k, Resistor_SMD:R_0603_1608Metric, B.Cu at (222.2, 150.1)
- added R14: 6k, Resistor_SMD:R_0603_1608Metric, B.Cu at (110.1, 67.2)
- added R15: 6k, Resistor_SMD:R_0603_1608Metric, B.Cu at (218.1, 132.6)
- added R16: 1k, Resistor_SMD:R_0603_1608Metric, B.Cu at (106.8, 65.5)
- added R17: 1k, Resistor_SMD:R_0603_1608Metric, B.Cu at (218.1, 137.6)
- added R18: 1k, Resistor_SMD:R_0603_1608Metric, B.Cu at (106.8, 63.2)
- added R19: 1k, Resistor_SMD:R_0603_1608Metric, B.Cu at (218.1, 142.6)
- added R2: 4.7k, Resistor_SMD:R_0603_1608Metric, B.Cu at (45.9, 37.5)
- added R20: 6k, Resistor_SMD:R_0603_1608Metric, B.Cu at (110.1, 61.5)
- added R21: 6k, Resistor_SMD:R_0603_1608Metric, B.Cu at (218.1, 147.6)
- added R22: 6k, Resistor_SMD:R_0603_1608Metric, B.Cu at (146.0, 67.3)
- added R23: 6k, Resistor_SMD:R_0603_1608Metric, B.Cu at (218.1, 152.7)
- added R24: 1k, Resistor_SMD:R_0603_1608Metric, B.Cu at (142.7, 65.7)
- added R25: 1k, Resistor_SMD:R_0603_1608Metric, B.Cu at (214.1, 135.1)
- added R26: 1k, Resistor_SMD:R_0603_1608Metric, B.Cu at (142.7, 63.4)
- added R27: 1k, Resistor_SMD:R_0603_1608Metric, B.Cu at (214.1, 140.1)
- added R28: 6k, Resistor_SMD:R_0603_1608Metric, B.Cu at (146.0, 61.6)
- added R29: 6k, Resistor_SMD:R_0603_1608Metric, B.Cu at (214.1, 145.1)
- added R3: 4.7k, Resistor_SMD:R_0603_1608Metric, B.Cu at (48.9, 37.5)
- added R30: 6k, Resistor_SMD:R_0603_1608Metric, B.Cu at (214.1, 147.6)
- added R31: 6k, Resistor_SMD:R_0603_1608Metric, B.Cu at (214.1, 150.1)
- added R32: 1k, Resistor_SMD:R_0603_1608Metric, B.Cu at (214.1, 152.7)
- added R33: 1k, Resistor_SMD:R_0603_1608Metric, B.Cu at (210.1, 132.6)
- added R34: 1k, Resistor_SMD:R_0603_1608Metric, B.Cu at (210.1, 135.1)
- added R35: 1k, Resistor_SMD:R_0603_1608Metric, B.Cu at (210.1, 137.6)
- added R36: 6k, Resistor_SMD:R_0603_1608Metric, B.Cu at (210.1, 140.1)
- added R41: 1k, Resistor_SMD:R_0603_1608Metric, B.Cu at (151.9, 65.3)
- added R42: 4k, Resistor_SMD:R_0603_1608Metric, B.Cu at (151.9, 66.8)
- added R43: 3.57k, Resistor_SMD:R_0603_1608Metric, B.Cu at (148.2, 47.8)
- added R44: 1.15k, Resistor_SMD:R_0603_1608Metric, B.Cu at (148.2, 49.4)
- added R6: 6k, Resistor_SMD:R_0603_1608Metric, B.Cu at (64.9, 69.7)
- added R7: 6k, Resistor_SMD:R_0603_1608Metric, B.Cu at (222.2, 135.1)
- added R8: 1k, Resistor_SMD:R_0603_1608Metric, B.Cu at (61.6, 68.0)
- added R9: 1k, Resistor_SMD:R_0603_1608Metric, B.Cu at (222.2, 140.1)
- C102: renamed from C12; footprint Capacitor_SMD:C_0603_1608Metric -> Capacitor_SMD:C_0805_2012Metric
- C109: renamed from C18; footprint Capacitor_SMD:C_0603_1608Metric -> Capacitor_SMD:C_0805_2012Metric
- C73: renamed from C37; footprint Capacitor_SMD:C_0402_1005Metric -> Capacitor_SMD:C_0603_1608Metric
- C74: renamed from C38; footprint Capacitor_SMD:C_0402_1005Metric -> Capacitor_SMD:C_0603_1608Metric
- C75: renamed from C39; footprint Capacitor_SMD:C_0402_1005Metric -> Capacitor_SMD:C_0603_1608Metric
- C76: renamed from C34; footprint Capacitor_SMD:C_0402_1005Metric -> Capacitor_SMD:C_0603_1608Metric
- C78: renamed from C35; footprint Capacitor_SMD:C_0402_1005Metric -> Capacitor_SMD:C_0603_1608Metric
- C79: renamed from C36; footprint Capacitor_SMD:C_0402_1005Metric -> Capacitor_SMD:C_0603_1608Metric
- C86: renamed from C40; value 100nf -> 1uf; footprint Capacitor_SMD:C_0402_1005Metric -> Capacitor_SMD:C_0603_1608Metric
- C87: renamed from C41; value 100nf -> 1uf; footprint Capacitor_SMD:C_0402_1005Metric -> Capacitor_SMD:C_0603_1608Metric
- C88: renamed from C42; value 100nf -> 1uf; footprint Capacitor_SMD:C_0402_1005Metric -> Capacitor_SMD:C_0603_1608Metric
- C89: renamed from C43; value 100nf -> 1uf; footprint Capacitor_SMD:C_0402_1005Metric -> Capacitor_SMD:C_0603_1608Metric
- C90: renamed from C44; value 100nf -> 1uf; footprint Capacitor_SMD:C_0402_1005Metric -> Capacitor_SMD:C_0603_1608Metric
- C91: renamed from C45; value 100nf -> 1uf; footprint Capacitor_SMD:C_0402_1005Metric -> Capacitor_SMD:C_0603_1608Metric
- C92: renamed from C46; value 100nf -> 1uf; footprint Capacitor_SMD:C_0402_1005Metric -> Capacitor_SMD:C_0603_1608Metric
- C93: renamed from C47; value 100nf -> 1uf; footprint Capacitor_SMD:C_0402_1005Metric -> Capacitor_SMD:C_0603_1608Metric
- C94: renamed from C13; footprint Capacitor_SMD:C_0603_1608Metric -> Capacitor_SMD:C_0805_2012Metric
- C95: renamed from C7; footprint Capacitor_SMD:C_0603_1608Metric -> Capacitor_SMD:C_0805_2012Metric
- R37: value 10k -> 6k
- moved C94 162.0 mm to (54.5, 47.5), turned to -90 degrees
- moved U19 159.6 mm to (51.6, 47.5), turned to 0 degrees
- moved C95 158.5 mm to (48.9, 47.5), turned to 90 degrees
- moved R40 157.1 mm to (57.9, 47.5), turned to 90 degrees
- moved C96 156.4 mm to (51.6, 50.1)
- moved R39 156.2 mm to (56.3, 47.5), turned to -90 degrees
- moved SW1 126.7 mm to (59.5, 78.0), turned to -90 degrees
- moved U10 126.2 mm to (65.0, 66.8), turned to 90 degrees
- moved C109 116.9 mm to (148.9, 44.9), turned to 90 degrees
- moved C111 108.7 mm to (151.7, 50.5), turned to 0 degrees
- moved C102 106.7 mm to (152.1, 60.2)
- moved C106 96.4 mm to (155.8, 67.8), turned to 0 degrees
- moved U12 90.8 mm to (110.1, 64.4), turned to 90 degrees
- moved U21 88.9 mm to (152.4, 47.5)
- moved U15 81.2 mm to (145.9, 64.5), turned to 90 degrees
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- renumbered C11 to C106, C17 to C111, C8 to C96, J1 to J2, R44 to R1, R40 to R39, R43 to R4, R41 to R40, R45 to R5, SW2 to SW1, U21 to U1, U9 to U10, U13 to U11, U10 to U12, U14 to U13, U17 to U14, U11 to U15, U15 to U16, U12 to U17, U16 to U18, U18 to U19, U1 to U2, U19 to U20, U20 to U21, U2 to U3, U3 to U4, U4 to U5, U5 to U6, U6 to U7, U7 to U8, U8 to U9
Connections:
- R37 pad 1: +5V -> Net-(U18--)
- R37 pad 2: Net-(U18-PG) -> /Analog/AIN_7P
- R4 pad 1: Net-(SW1-B) -> GND
- U18 pad 4: Net-(U16--) (its old number) -> Net-(U18--)
- U19 pad 7: Net-(U18-PG) -> unconnected-(U19-PG-Pad7)
