File: MW601_KB.kicad_sch (KiCad schematic)
At the start: 0 parts

Commit message: sch
Parts:
- added H1, H2, H3, H4, H5, H6: MountingHole_Pad, symbol Mechanical:MountingHole_Pad
- added H10: Stabilizer_Cherry_MX_6.25u, symbol Mechanical:MountingHole
- added H7, H8, H9: Stabilizer_Cherry_MX_2.00u, symbol Mechanical:MountingHole
Connections:
- new net GND: H1.1, H2.1, H3.1, H4.1, H5.1, H6.1
Other:
- added sheet Analog (Analog.kicad_sch)
- added sheet Power Supply (power.kicad_sch)
- sheet Key Layout ports: added LED_SDA, {Matrix_OUT}; removed none
- sheet MCU ports: added A0, A1, A2, EN, LED_SDA, SPI1_MISO, SPI1_MOSI, SPI1_NSS, SPI1_SCK, ~{RST/PD}; removed none
- sheet TMUX ports: added A0, A1, A2, EN, GP0_OUT+, GP0_OUT-, GP1_OUT+, GP1_OUT-, GP2_OUT+, GP2_OUT-, GP3_OUT+, GP3_OUT-, GP4_OUT+, GP4_OUT-, GP5_OUT+, GP5_OUT-, GP6_OUT+, GP6_OUT-, GP7_OUT+, GP7_OUT-, {Matrix_OUT}; removed none

Commit message: add cap
Parts:
- H1: footprint (none) -> hole:PKRHC
- H10: footprint (none) -> PCM_Mounting_Keyboard_Stabilizer:Stabilizer_Cherry_MX_6.25u
- H2, H3, H6: footprint (none) -> hole:PKRH
- H4, H5: footprint (none) -> hole:PKRHSL
- H7, H8, H9: footprint (none) -> PCM_Mounting_Keyboard_Stabilizer:Stabilizer_Cherry_MX_2.00u
Changed lines of the file:
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@@
 			)
 		)
-		(property "Footprint" ""
+		(property "Footprint" "hole:PKRHSL"
 			(at 274.32 63.5 0)
 			(effects
@@
 			)
 		)
-		(property "Footprint" ""
+		(property "Footprint" "hole:PKRHSL"
 			(at 274.32 53.34 0)
 			(effects
@@
 			)
 		)
-		(property "Footprint" ""
+		(property "Footprint" "PCM_Mounting_Keyboard_Stabilizer:Stabilizer_Cherry_MX_2.00u"
 			(at 231.14 24.13 0)
 			(effects
@@
 		(dnp no)
 		(fields_autoplaced yes)
-		(property "Reference" "#PWR0135"
+		(property "Reference" "#PWR01"
 			(at 276.86 83.82 0)
 			(effects
@@
 			(project ""
 				(path "/646e296e-2dfc-4fd5-a15b-e5e3814d0740"
-					(reference "#PWR0135")
+					(reference "#PWR01")
 					(unit 1)
 				)
@@
 			)
 		)
-		(property "Footprint" ""
+		(property "Footprint" "hole:PKRH"
 			(at 274.32 73.66 0)
 			(effects
@@
 			)
 		)
-		(property "Footprint" ""
+		(property "Footprint" "PCM_Mounting_Keyboard_Stabilizer:Stabilizer_Cherry_MX_6.25u"
 			(at 231.14 34.29 0)
 			(effects
@@
 			)
 		)
-		(property "Footprint" ""
+		(property "Footprint" "hole:PKRH"
 			(at 274.32 33.02 0)
 			(effects
@@
 			)
 		)
-		(property "Footprint" ""
+		(property "Footprint" "hole:PKRH"
 			(at 274.32 43.18 0)
 			(effects
@@
 			)
 		)
-		(property "Footprint" ""
+		(property "Footprint" "PCM_Mounting_Keyboard_Stabilizer:Stabilizer_Cherry_MX_2.00u"
 			(at 231.14 29.21 0)
 			(effects
@@
 			)
 		)
-		(property "Footprint" ""
+		(property "Footprint" "PCM_Mounting_Keyboard_Stabilizer:Stabilizer_Cherry_MX_2.00u"
 			(at 231.14 19.05 0)
 			(effects
@@
 			)
 		)
-		(property "Footprint" ""
+		(property "Footprint" "hole:PKRHC"
 			(at 274.32 22.86 0)
 			(effects
