File: layout.kicad_sch (KiCad schematic)
At the start: 128 parts

Commit message: sch
Parts:
- added C21, C22, C23, C24, C25, C26, C27, C28: 47uf, symbol Device:C_Small
Connections:
- net GND: now also C21.2, C22.2, C23.2, C24.2, C25.2, C26.2, C27.2, C28.2
- net VCC_LED renamed +5V
- net +5V: now also C21.1, C22.1, C23.1, C24.1, C25.1, C26.1, C27.1, C28.1
- net VSSA renamed VCC1V0

Commit message: add cap
Parts:
- added C1, C10, C11, C12, C13, C14, C15, C16, C17, C18, C19, C2, C20, C21, C22, C23, C24, C25, C26, C27, C28, C29, C3, C30, C31, C32, C33, C34, C35, C36, C37, C38, C39, C4, C40, C41, C42, C43, C44, C45, C46, C47, C48, C49, C5, C50, C51, C52, C53, C54, C55, C56, C57, C58, C59, C6, C60, C61, C62, C63, C64, C7, C8, C9: 1uf, Capacitor_SMD:C_0603_1608Metric, symbol Device:C_Small
- C65: renamed from C21; footprint (none) -> Capacitor_SMD:C_0805_2012Metric
- C66: renamed from C22; footprint (none) -> Capacitor_SMD:C_0805_2012Metric
- C67: renamed from C23; footprint (none) -> Capacitor_SMD:C_0805_2012Metric
- C68: renamed from C24; footprint (none) -> Capacitor_SMD:C_0805_2012Metric
- C69: renamed from C25; footprint (none) -> Capacitor_SMD:C_0805_2012Metric
- C70: renamed from C26; footprint (none) -> Capacitor_SMD:C_0805_2012Metric
- C71: renamed from C27; footprint (none) -> Capacitor_SMD:C_0805_2012Metric
- C72: renamed from C28; footprint (none) -> Capacitor_SMD:C_0805_2012Metric
Connections:
- net GND: now also C1.2, C10.2, C11.2, C12.2, C13.2, C14.2, C15.2, C16.2, C17.2, C18.2, C19.2, C2.2, C20.2, C21.2, C22.2, C23.2, C24.2, C25.2, C26.2, C27.2, C28.2, C29.2, C3.2, C30.2, C31.2, C32.2, C33.2, C34.2, C35.2, C36.2, C37.2, C38.2, C39.2, C4.2, C40.2, C41.2, C42.2, C43.2, C44.2, C45.2, C46.2, C47.2, C48.2, C49.2, C5.2, C50.2, C51.2, C52.2, C53.2, C54.2, C55.2, C56.2, C57.2, C58.2, C59.2, C6.2, C60.2, C61.2, C62.2, C63.2, C64.2, C7.2, C8.2, C9.2
- net VCC1V0: now also C1.1, C10.1, C11.1, C12.1, C13.1, C14.1, C15.1, C16.1, C17.1, C18.1, C19.1, C2.1, C20.1, C21.1, C22.1, C23.1, C24.1, C25.1, C26.1, C27.1, C28.1, C29.1, C3.1, C30.1, C31.1, C32.1, C33.1, C34.1, C35.1, C36.1, C37.1, C38.1, C39.1, C4.1, C40.1, C41.1, C42.1, C43.1, C44.1, C45.1, C46.1, C47.1, C48.1, C49.1, C5.1, C50.1, C51.1, C52.1, C53.1, C54.1, C55.1, C56.1, C57.1, C58.1, C59.1, C6.1, C60.1, C61.1, C62.1, C63.1, C64.1, C7.1, C8.1, C9.1
Other:
- moved on the sheet: C65, C66, C67, C68, C69, C70, C71, C72
