File: power.kicad_sch (KiCad schematic)
At the start: 28 parts, among them U18 TPS82130, U19 TPS74801DRC, U20 TPS74801DRC

Commit message: add cap
Parts:
- removed R37: 10k, Resistor_SMD:R_0603_1608Metric, symbol Device:R_Small
- C100: renamed from C10; footprint (none) -> Capacitor_SMD:C_0603_1608Metric
- C101: renamed from C31; footprint (none) -> Capacitor_SMD:C_0603_1608Metric
- C102: renamed from C12; footprint Capacitor_SMD:C_0603_1608Metric -> Capacitor_SMD:C_0805_2012Metric
- C103: renamed from C14; footprint (none) -> Capacitor_SMD:C_0805_2012Metric
- C104: renamed from C33; footprint (none) -> Capacitor_SMD:C_0603_1608Metric
- C105: renamed from C32; footprint (none) -> Capacitor_SMD:C_0603_1608Metric
- C107: renamed from C15; footprint (none) -> Capacitor_SMD:C_0603_1608Metric
- C108: renamed from C16; footprint (none) -> Capacitor_SMD:C_0603_1608Metric
- C109: renamed from C18; footprint Capacitor_SMD:C_0603_1608Metric -> Capacitor_SMD:C_0805_2012Metric
- C110: renamed from C19; footprint (none) -> Capacitor_SMD:C_0805_2012Metric
- C94: renamed from C13; footprint Capacitor_SMD:C_0603_1608Metric -> Capacitor_SMD:C_0805_2012Metric
- C95: renamed from C7; footprint Capacitor_SMD:C_0603_1608Metric -> Capacitor_SMD:C_0805_2012Metric
- C97: renamed from C9; footprint (none) -> Capacitor_SMD:C_0603_1608Metric
- C98: renamed from C29; footprint (none) -> Capacitor_SMD:C_0805_2012Metric
- C99: renamed from C30; footprint (none) -> Capacitor_SMD:C_0805_2012Metric
- R41: renamed from R35; footprint (none) -> Resistor_SMD:R_0603_1608Metric
- R42: renamed from R36; footprint (none) -> Resistor_SMD:R_0603_1608Metric
- R43: renamed from R38; footprint (none) -> Resistor_SMD:R_0603_1608Metric
- R44: renamed from R39; footprint (none) -> Resistor_SMD:R_0603_1608Metric
- renumbered C11 to C106, C17 to C111, C8 to C96, R40 to R39, R41 to R40, U18 to U19, U19 to U20, U20 to U21
Connections:
- no-connect marks 2 -> 3
