File: mcu.kicad_sch (KiCad schematic)
At the start: 1 part, among them J1 USB_C_Receptacle_USB2.0_16P

Commit message: sch
Parts:
- added C20: 47uf Polarized, symbol Device:C_Polarized
- added C34, C37, C38, C39: 100nf, Capacitor_SMD:C_0402_1005Metric, symbol Device:C
- added C35, C36: 12pf, Capacitor_SMD:C_0402_1005Metric, symbol Device:C
- added D65: LED, symbol Device:LED
- added J2: Conn_01x06, symbol Connector_Generic:Conn_01x06
- added R33, R34: 4.7k, symbol Device:R_Small
- added R43, R44: 4.7k, Resistor_SMD:R_0603_1608Metric, symbol Device:R
- added R45: 510R, Resistor_SMD:R_0603_1608Metric, symbol Device:R
- added SW1: SW_SPDT, Button_Switch_THT:SW_Slide_SPDT_Straight_CK_OS102011MS2Q, symbol Switch:SW_SPDT
- added SW2: SW_Push, Button_Switch_SMD:SW_Push_1P1T_XKB_TS-1187A, symbol Switch:SW_Push
- added U21: CH32V30xCxTx, Package_QFP:LQFP-48_7x7mm_P0.5mm, symbol MCU_WCH_CH32V3:CH32V30xCxTx
- added Y1: Crystal_GND24, Crystal:Crystal_SMD_3225-4Pin_3.2x2.5mm, symbol Device:Crystal_GND24
Connections:
- net GND: now reaches J1.A1 (GND), J1.A12 (GND), J1.B1 (GND), J1.B12 (GND)
- net GND: now also J1.S1 (SHIELD), C20.2, C34.1, C35.1, C36.1, C37.1, C38.1, C39.1, J2.6 (Pin_6), R33.2, R34.2, SW1.3 (C), SW2.1, U21.23 (VSS), U21.35 (VSS), U21.47 (VSS), U21.8 (VSSA), Y1.2, Y1.4
- net +5V: now reaches J1.A4 (VBUS), J1.A9 (VBUS), J1.B4 (VBUS), J1.B9 (VBUS)
- net +5V: now also C20.1
- net at J1.A5 (CC1): now also R33.1
- net D+: now reaches J1.A6 (D+)
- net D+: now also J1.B6 (D+), U21.43 (PB7)
- net D-: now reaches J1.A7 (D-)
- net D-: now also J1.B7 (D-), U21.42 (PB6)
- net at J1.B5 (CC2): now also R34.1
- new net: D65.1 (K), U21.28 (PB15)
- new net: D65.2 (A), R45.1
- new net: R43.1, SW1.2 (B)
- new net +3V3: C37.2, C38.2, C39.2, J2.1 (Pin_1), R44.2, R45.2, SW1.1 (A), U21.1 (VBAT), U21.24 (VDD), U21.36 (VDD), U21.48 (VDD), U21.9 (VDDA)
- new net A0: U21.18 (PB0)
- new net A1: U21.19 (PB1)
- new net A2: U21.20 (PB2)
- new net BOOT0: R43.2, U21.44 (BOOT0)
- new net EN: U21.39 (PB3)
- new net LED_SDA: U21.29 (PA8)
- new net NRST: C34.2, R44.1, SW2.2, U21.7 (~{RST})
- new net OSC_IN: C35.2, U21.5 (OSC_IN), Y1.3
- new net OSC_OUT: C36.2, U21.6 (OSC_OUT), Y1.1
- new net SPI1_MISO: U21.16 (PA6)
- new net SPI1_MOSI: U21.17 (PA7)
- new net SPI1_NSS: U21.14 (PA4)
- new net SPI1_SCK: U21.15 (PA5)
- new net SWCLK: J2.3 (Pin_3), U21.37 (SWCLK)
- new net SWDIO: J2.2 (Pin_2), U21.34 (SWDIO)
- new net USART1_RX: J2.5 (Pin_5), U21.31 (PA10)
- new net USART1_TX: J2.4 (Pin_4), U21.30 (PA9)
- new net ~{RST/PD}: U21.13 (PA3)
- no-connect marks 0 -> 20
Other:
- moved on the sheet: J1

Commit message: add cap
Parts:
- removed SW1: SW_SPDT, Button_Switch_THT:SW_Slide_SPDT_Straight_CK_OS102011MS2Q, symbol Switch:SW_SPDT
- added J3: Boot0, Connector_PinHeader_2.54mm:PinHeader_1x02_P2.54mm_Vertical, symbol Connector_Generic:Conn_01x02
- C73: renamed from C37; footprint Capacitor_SMD:C_0402_1005Metric -> Capacitor_SMD:C_0603_1608Metric
- C74: renamed from C38; footprint Capacitor_SMD:C_0402_1005Metric -> Capacitor_SMD:C_0603_1608Metric
- C75: renamed from C39; footprint Capacitor_SMD:C_0402_1005Metric -> Capacitor_SMD:C_0603_1608Metric
- C76: renamed from C34; footprint Capacitor_SMD:C_0402_1005Metric -> Capacitor_SMD:C_0603_1608Metric
- C77: renamed from C20; footprint (none) -> Capacitor_Tantalum_SMD:CP_EIA-3528-21_Kemet-B
- C78: renamed from C35; footprint Capacitor_SMD:C_0402_1005Metric -> Capacitor_SMD:C_0603_1608Metric
- C79: renamed from C36; footprint Capacitor_SMD:C_0402_1005Metric -> Capacitor_SMD:C_0603_1608Metric
- D65: footprint (none) -> LED_SMD:LED_0603_1608Metric
- J1: renamed from J2; footprint (none) -> Connector_PinHeader_2.54mm:PinHeader_1x06_P2.54mm_Vertical
- R2: renamed from R33; footprint (none) -> Resistor_SMD:R_0603_1608Metric
- R3: renamed from R34; footprint (none) -> Resistor_SMD:R_0603_1608Metric
- renumbered J1 to J2, R44 to R1, R43 to R4, R45 to R5, SW2 to SW1, U21 to U1
Connections:
- net +3V3: now also J3.1 (Pin_1)
- net BOOT0: now also J3.2 (Pin_2)
- net GND: now also R4.1
Other:
- moved on the sheet: R4

Commit message: solder
Parts:
- removed U1: CH32V30xCxTx, Package_QFP:LQFP-48_7x7mm_P0.5mm, symbol MCU_WCH_CH32V3:CH32V30xCxTx
- added C112, C113, C114: 100nf, Capacitor_SMD:C_0603_1608Metric, symbol Device:C
- added R38: 4.7k, Resistor_SMD:R_0603_1608Metric, symbol Device:R
- added U22: W25Q128JVS, Package_SO:SOIC-8_5.23x5.23mm_P1.27mm, symbol Memory_Flash:W25Q128JVS
- added U23: CH32V30xRxTx, Package_QFP:LQFP-64_10x10mm_P0.5mm, symbol MCU_WCH_CH32V3:CH32V30xRxTx
Connections:
- net +3V3: now also C112.2, C113.2, C114.2, R38.2, U22.8 (VCC), U23.1 (VBAT), U23.13 (VDDA), U23.19 (VDD), U23.32 (VIO), U23.48 (VDD), U23.64 (VIO)
- net A0: now also U23.26 (PB0)
- net A1: now also U23.27 (PB1)
- net A2: now also U23.28 (PB2)
- net BOOT0: now also U23.60 (BOOT0)
- net D+: now also U23.59 (PB7)
- net D-: now also U23.58 (PB6)
- net EN: now also U23.55 (PB3)
- net GND: now also C112.1, C113.1, C114.1, U22.4 (GND), U23.12 (VSSA), U23.18 (VSS), U23.31 (VSS), U23.47 (VSS), U23.63 (VSS)
- net LED_SDA: now also U23.41 (PA8)
- net NRST: now also U23.7 (~{RST})
- net OSC_IN: now also U23.5 (OSC_IN)
- net OSC_OUT: now also U23.6 (OSC_OUT)
- net SPI1_MISO: now also U23.22 (PA6)
- net SPI1_MOSI: now also U23.23 (PA7)
- net SPI1_NSS: now also U23.20 (PA4)
- net SPI1_SCK: now also U23.21 (PA5)
- net SWCLK: now also U23.49 (SWCLK)
- net SWDIO: now also U23.46 (SWDIO)
- net USART1_RX: now also U23.43 (PA10)
- net USART1_TX: now also U23.42 (PA9)
- net ~{RST/PD}: now also U23.17 (PA3)
- net LED_Pin: now reaches D65.1 (K)
- net LED_Pin: now also U23.14 (PA0)
- new net SPI2_MISO: U22.2 (DO(IO1)), U23.35 (PB14)
- new net SPI2_MOSI: U22.5 (DI(IO0)), U23.36 (PB15)
- new net SPI2_NSS: R38.1, U22.1 (~{CS}), U23.33 (PB12)
- new net SPI2_SCK: U22.6 (CLK), U23.34 (PB13)
- no-connect marks 20 -> 32
Other:
- note added: "EEPROM"
- note added: "LED"
- note added: "USB"
- moved on the sheet: C76, C77, C78, C79, D65, J2, J3, R1, R2, R3, R4, R5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
